File: bottom/Nixieclock.sch (EAGLE design)
At the start: 59 parts, among them IC1 R-78E5.0-0.5, SW1 AL1, SW2 AL2, SW3 UP, SW4 DN, T1 MPSA42, T2 MPSA42, T8 IRF640N, T9 BC516, U1 MC33063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

Commit message: Updated schematic
Parts:
- U1: value MC33063 -> MC34063
Changed lines of the file:
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@@
 <layer number="230" name="230bmp" color="7" fill="1" visible="yes" active="yes"/>
 <layer number="231" name="231bmp" color="7" fill="1" visible="yes" active="yes"/>
+<layer number="232" name="Eagle3D_PG2" color="7" fill="1" visible="no" active="no"/>
+<layer number="233" name="Eagle3D_PG3" color="7" fill="1" visible="no" active="no"/>
 <layer number="248" name="Housing" color="7" fill="1" visible="yes" active="yes"/>
 <layer number="249" name="Edge" color="7" fill="1" visible="yes" active="yes"/>
@@
 <part name="R20" library="resistor" deviceset="R-EU_" device="0207/10" value="560K"/>
 <part name="D3" library="diode" deviceset="1N4004" device="" value="SB140"/>
-<part name="U1" library="adafruit" deviceset="MC33063/MC34063" device="P" value="MC33063"/>
+<part name="U1" library="adafruit" deviceset="MC33063/MC34063" device="P" value="MC34063"/>
 <part name="GND7" library="supply1" deviceset="GND" device=""/>
 <part name="GND8" library="supply1" deviceset="GND" device=""/>
